Commit message: updated working model

File: Quadruped_sim/urdf/Quadruped.urdf (robot description, URDF)
Before this commit: robot Quadruped2, 13 links, 12 joints
Links:
- link base_link: mass 0.2676 -> 0.267600954992518
- link leg_1_hip: mass 0.067078 -> 0.067077762894934
- link leg_1_knee: mass 0.0696914929566026 -> 0.0696914928060746
- link leg_2_hip: mass 0.067077752877841 -> 0.0670777528778422
- link leg_2_knee: mass 0.0696914931210686 -> 0.0696914931210657
- link leg_3_ankle: mass 0.0169824099129692 -> 0.0169824099129693
- link leg_3_hip: mass 0.066276459588986 -> 0.0662764719650818
- link leg_3_knee: mass 0.0696914931416134 -> 0.0696914925297254
- link leg_4_ankle: mass 0.0169824099129692 -> 0.0169824099129693
- link leg_4_hip: mass 0 -> 0.0662764580966196
- link leg_4_knee: mass 0.0696914932488965 -> 0.0696914932488991
Joints:
- joint leg1_hip_joint: limit lower=0 upper=0 effort=10 velocity=5 -> lower=0 upper=3 effort=10 velocity=5; origin xyz=0.06197 -0.082557 0.0385 rpy=-3.1416 0 -0.11014 -> xyz=0.06197 -0.082557 0.0385 rpy=3.1416 0 -0.056054
- joint leg_1_ankle_joint: limit lower=0 upper=0 effort=10 velocity=5 -> lower=0 upper=3 effort=10 velocity=5; origin xyz=-0.026724 0.0005 -0.059001 rpy=3.1416 -1.0269 -3.1416 -> xyz=-0.046499 0.0005 -0.045091 rpy=3.1416 -1.0269 -3.1416
- joint leg_1_knee_joint: limit lower=0 upper=0 effort=10 velocity=5 -> lower=0 upper=3 effort=10 velocity=5
- joint leg_2_ankle_joint: limit lower=0 upper=0 effort=10 velocity=5 -> lower=0 upper=3 effort=10 velocity=5
- joint leg_2_hip_joint: limit lower=0 upper=0 effort=10 velocity=5 -> lower=0 upper=3 effort=10 velocity=5; origin xyz=0.06177 0.0055571 0.0385 rpy=3.1416 0 0.85297 -> xyz=0.06177 0.0055571 0.0385 rpy=3.1416 0 0.90705
- joint leg_2_knee_joint: limit lower=0 upper=0 effort=10 velocity=5 -> lower=0 upper=3 effort=10 velocity=5
- joint leg_3_ankle: limit lower=0 upper=0 effort=10 velocity=5 -> lower=0 upper=3 effort=10 velocity=5
- joint leg_3_hip_joint: limit lower=0 upper=0 effort=10 velocity=5 -> lower=0 upper=3 effort=10 velocity=5; origin xyz=-0.04277 0.0055571 0.0395 rpy=3.1416 0 2.8191 -> xyz=-0.04277 0.0055571 0.0395 rpy=-3.1416 0 -2.9812
- joint leg_3_knee_joint: limit lower=0 upper=0 effort=10 velocity=5 -> lower=0 upper=3 effort=10 velocity=5
- joint leg_4_ankle_joint: limit lower=0 upper=0 effort=10 velocity=5 -> lower=0 upper=3 effort=10 velocity=5
- joint leg_4_hip_joint: limit lower=0 upper=0 effort=10 velocity=5 -> lower=0 upper=3 effort=10 velocity=5; origin xyz=-0.04277 -0.082557 0.0385 rpy=3.1416 0 2.7272 -> xyz=-0.04277 -0.082557 0.0385 rpy=-3.1416 0 2.7813
- joint leg_4_knee_joint: limit lower=0 upper=0 effort=10 velocity=5 -> lower=0 upper=3 effort=10 velocity=5
