Commit message: Update PressTip2.urdf

File: Quadruped_sim/PressTip2/urdf/PressTip2.urdf (robot description, URDF)
Before this commit: robot PressTip2, 17 links, 16 joints
Links:
- link base_link: geometry collision mesh filename=meshes/base_link.STL; visual mesh filename=meshes/base_link.STL
- link leg1foot: geometry collision mesh filename=meshes/leg1foot.STL; visual mesh filename=meshes/leg1foot.STL
- link leg1hip: geometry collision mesh filename=meshes/leg1hip.STL; visual mesh filename=meshes/leg1hip.STL
- link leg1knee: geometry collision mesh filename=meshes/leg1knee.STL; visual mesh filename=meshes/leg1knee.STL
- link leg2foot: geometry collision mesh filename=meshes/leg2foot.STL; visual mesh filename=meshes/leg2foot.STL
- link leg2hip: geometry collision mesh filename=meshes/leg2hip.STL; visual mesh filename=meshes/leg2hip.STL
- link leg2knee: geometry collision mesh filename=meshes/leg2knee.STL; visual mesh filename=meshes/leg2knee.STL
- link leg3foot: geometry collision mesh filename=meshes/leg3foot.STL; visual mesh filename=meshes/leg3foot.STL
- link leg3hip: geometry collision mesh filename=meshes/leg3hip.STL; visual mesh filename=meshes/leg3hip.STL
- link leg3knee: geometry collision mesh filename=meshes/leg3knee.STL; visual mesh filename=meshes/leg3knee.STL
- link leg4foot: geometry collision mesh filename=meshes/leg4foot.STL; visual mesh filename=meshes/leg4foot.STL
- link leg4hip: geometry collision mesh filename=meshes/leg4hip.STL; visual mesh filename=meshes/leg4hip.STL
- link leg4knee: geometry collision mesh filename=meshes/leg4knee.STL; visual mesh filename=meshes/leg4knee.STL
- link tip1: geometry collision mesh filename=meshes/tip1.STL; visual mesh filename=meshes/tip1.STL
- link tip2: geometry collision mesh filename=meshes/tip2.STL; visual mesh filename=meshes/tip2.STL
- link tip3: geometry collision mesh filename=meshes/tip3.STL; visual mesh filename=meshes/tip3.STL
- link tip4: geometry collision mesh filename=meshes/tip4.STL; visual mesh filename=meshes/tip4.STL
